File: hardware/KiCAD/Pronoia_Sustainer/Power.kicad_sch (KiCad schematic)
At the start: 17 parts, among them J1 XT30PW-M, J2 Screw_Terminal_01x02, U1 TPS563201, U3 AP2112K-3.3

Commit message: updated Schematics
Other:
- note added: "2S LiPo Voltage Monitor"
- note removed: "Voltage Monitor"
Changed lines of the file:
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@@
 	(text "5 V Buck Converter"
 		(exclude_from_sim no)
-		(at 113.284 68.326 0)
+		(at 122.428 68.072 0)
 		(effects
 			(font
@@
 		)
 	)
-	(text "Voltage Monitor"
+	(text "2S LiPo Voltage Monitor"
 		(exclude_from_sim no)
 		(at 226.568 78.74 0)

Commit message: Completed 1st draft of Schematic
Other:
- note added: "2S 8.4 V LiPo Battery XT30 Connection"
- note added: "Rotary Key Switch Screw Terminal Block Conn"
- note removed: "2S 8.4 V LiPo Battery"
- note removed: "Rotary Key Switch"
- moved on the sheet: J1, NT1

Commit message: Last commit for KiCAD schematic w/ GPS, Telem, and Bluetooth
Other:
- company: (none) -> Walla Walla University
- title: (none) -> Pronoia Sustainer Power Management
Changed lines of the file:
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@@
 	(generator_version "9.0")
 	(paper "A4")
+	(title_block
+		(title "Pronoia Sustainer Power Management")
+		(date "2026-02-03")
+		(rev "1.0")
+		(company "Walla Walla University")
+		(comment 1 "Prometheus Rocket Project")
+	)
 	(text "3.3V LDO Regulator"
 		(exclude_from_sim no)

Commit message: Finalized v2.0 of Pronoia Schematic
Parts:
- removed C7, C8: 1uF, PCM_JLCPCB:C_0603, symbol PCM_JLCPCB-Capacitors:0603,1uF
- removed NT1: NetTie_2, NetTie:NetTie-2_SMD_Pad2.0mm, symbol Device:NetTie_2
- removed U3: AP2112K-3.3, Package_TO_SOT_SMD:SOT-23-5, symbol Regulator_Linear:AP2112K-3.3
- added C8: 100nF, PCM_JLCPCB:C_0402, symbol PCM_JLCPCB-Capacitors:0402,100nF
- J1: LCSC (none) -> C431092
- J2: now not fitted
Connections:
- net GNDPWR is gone; now on net GND: J1.N
- net GND: now also C8.2
- net Vbatt_Monitor: now also C8.1
- net +8.4V_ARMED: now reaches J2.2 (Pin_2)
- net +8.4V_ARMED: no longer J1.P
- net Vbatt_Post-Switch renamed +8.4V_LOGIC
- net +8.4V_LOGIC: now also J1.P
Other:
- note added: "FingerTech Mini Power Switch (Order and Connect via Terminal Screw Block)"
- note added: "FingerTech Mini Power Switch 5.08 mm Screw Terminal Block Conn"
- note added: "High Current Devices should be placed on one side of the board w/ low level logic components on the other side of the board. (The distinction between PWR_Ground and Signal Ground has been removed in v2.0)"
- note added: "Parts Not Shown/Notes"
- note removed: "3.3V LDO Regulator"
- note removed: "Parts Not Shown"
- note removed: "Rotary Key Switch (Order and Connect via Terminal Screw Block)"
- note removed: "Rotary Key Switch Screw Terminal Block Conn"

Commit message: Finished PCB layout
Parts:
- removed R1: 49.9kΩ, PCM_JLCPCB:R_0805, symbol PCM_JLCPCB-Resistors:0805,49.9kΩ
- removed R2: 9.1kΩ, PCM_JLCPCB:R_0805, symbol PCM_JLCPCB-Resistors:0805,9.1kΩ
- added R1: 56kΩ, PCM_JLCPCB:R_0603, symbol PCM_JLCPCB-Resistors:0603,56kΩ
- added R2: 10kΩ, PCM_JLCPCB:R_0603, symbol PCM_JLCPCB-Resistors:0603,10kΩ
Connections:
- net +5V: now also R1.1
- net GND: now also R2.2
- net at U1.4 (VFB): now also R1.2, R2.1

Commit message: Sensor Bring-Up
Parts:
- J2: now left out of the parts list
