File: hardware/KiCAD/Pronoia_Sustainer/Pronoia_Sustainer.kicad_pcb (KiCad board)
At the start: 2 copper layers, 0 parts

Commit message: Finished PCB layout
Parts:
- added BUZZER1: GSD9605YB-3V2800, GSD9605YB-3V2800:BUZ-SMD_GSD9605YB-3V2800, F.Cu at (118.1, 95.8)
- added C1: 10uF, PCM_JLCPCB:C_1206, F.Cu at (142.6, 145.8)
- added C10: 100nF, PCM_JLCPCB:C_0402, F.Cu at (141.0, 86.4)
- added C11: 100nF, PCM_JLCPCB:C_0402, F.Cu at (119.7, 77.2)
- added C12: 100nF, PCM_JLCPCB:C_0402, F.Cu at (135.0, 99.8)
- added C13: 100nF, PCM_JLCPCB:C_0402, F.Cu at (136.0, 96.0)
- added C14: 22uF, PCM_JLCPCB:C_0805, F.Cu at (147.8, 72.0)
- added C15: 100nF, PCM_JLCPCB:C_0402, F.Cu at (129.9, 140.0)
- added C16: 100nF, PCM_JLCPCB:C_0402, F.Cu at (129.8, 147.0)
- added C17: 100nF, PCM_JLCPCB:C_0402, F.Cu at (129.4, 154.6)
- added C18: 1000 uF, EEE-FT1A102AP, Capacitor_SMD:CP_Elec_8x10.5, F.Cu at (118.8, 120.9)
- added C19: 10uF, PCM_JLCPCB:C_1206, F.Cu at (152.0, 70.8)
- added C2: 10uF, PCM_JLCPCB:C_1206, F.Cu at (145.0, 145.8)
- added C20: 100nF, PCM_JLCPCB:C_0402, F.Cu at (148.2, 69.3)
- added C3: 22uF, PCM_JLCPCB:C_0805, F.Cu at (143.1, 142.0)
- added C4: 22uF, PCM_JLCPCB:C_0805, F.Cu at (143.1, 139.8)
- added C5: 100nF, PCM_JLCPCB:C_1206, F.Cu at (149.0, 141.4)
- added C6: 1000 uF, EEE-FT1A102AP, Capacitor_SMD:CP_Elec_8x10.5, F.Cu at (136.4, 147.8)
- added C7: 100nF, PCM_JLCPCB:C_0402, F.Cu at (129.4, 133.6)
- added C8: 100nF, PCM_JLCPCB:C_0402, F.Cu at (158.6, 155.4)
- added C9: 100nF, PCM_JLCPCB:C_0402, F.Cu at (138.2, 87.6)
- added D1: SS14, PCM_JLCPCB:D_SMA, F.Cu at (125.6, 132.0)
- added D2: SS14, PCM_JLCPCB:D_SMA, F.Cu at (125.6, 139.2)
- added D3: SS14, PCM_JLCPCB:D_SMA, F.Cu at (125.6, 146.4)
- added D4: SS14, PCM_JLCPCB:D_SMA, F.Cu at (125.6, 153.6)
- added D7: SS14, PCM_JLCPCB:D_SMA, F.Cu at (123.1, 103.2)
- added D8: LED, LED_SMD:LED_0603_1608Metric, F.Cu at (117.1, 85.4)
- added G***: LOGO, Graphics:IEEE Blue Logo, F.Cu at (174.8, 83.8)
- added G***: LOGO, Graphics:WWU Logo Horizontal, B.Cu at (116.2, 89.6)
- added J1: XT30PW-M, XT30PW-M:AMASS_XT30PW-M, F.Cu at (148.6, 162.8)
- added J11: 640457-2, 640457-2:TE_640457-2, F.Cu at (152.0, 125.3)
- added J12: Conn_01x24_Pin, Connector_PinSocket_2.54mm:PinSocket_1x24_P2.54mm_Vertical, F.Cu at (129.6, 68.0)
- added J14: Conn_01x24_Pin, Connector_PinSocket_2.54mm:PinSocket_1x24_P2.54mm_Vertical, F.Cu at (144.8, 68.0)
- added J2: Screw_Terminal_01x02, TerminalBlock_Phoenix:TerminalBlock_Phoenix_MKDS-1,5-2-5.08_1x02_P5.08mm_Horizontal, F.Cu at (157.2, 147.3)
- added J3: 1751303, 1751303:1751303, F.Cu at (116.6, 132.1)
- added J4: Servo0, Connector_PinHeader_2.54mm:PinHeader_1x03_P2.54mm_Vertical, F.Cu at (129.0, 164.3)
- added J5: Servo0, Connector_PinHeader_2.54mm:PinHeader_1x03_P2.54mm_Vertical, F.Cu at (132.6, 164.3)
- added J6: Servo0, Connector_PinHeader_2.54mm:PinHeader_1x03_P2.54mm_Vertical, F.Cu at (136.2, 164.3)
- added J7: Servo0, Connector_PinHeader_2.54mm:PinHeader_1x03_P2.54mm_Vertical, F.Cu at (139.8, 164.3)
- added J8: 640457-4, 640457-4:TE_640457-4, F.Cu at (148.1, 86.1)
- added L1: 3.3uH, Inductor_SMD:L_Bourns-SRN8040_8x8.15mm, F.Cu at (146.2, 133.4)
- added Q1: AO3400A, PCM_JLCPCB:Q_SOT-23, F.Cu at (129.6, 130.8)
- added Q2: AO3400A, PCM_JLCPCB:Q_SOT-23, F.Cu at (129.6, 137.4)
- added Q3: AO3400A, PCM_JLCPCB:Q_SOT-23, F.Cu at (129.7, 144.6)
- added Q4: AO3400A, PCM_JLCPCB:Q_SOT-23, F.Cu at (129.5, 151.8)
- added Q5: AO3400A, PCM_JLCPCB:Q_SOT-23, F.Cu at (155.3, 121.8)
- added Q6: AO3400A, PCM_JLCPCB:Q_SOT-23, F.Cu at (125.0, 97.9)
- added R1: 56kΩ, PCM_JLCPCB:R_0603, F.Cu at (153.0, 135.5)
- added R10: 10kΩ, PCM_JLCPCB:R_0805, F.Cu at (141.2, 119.0)
- added R11: 100Ω, PCM_JLCPCB:R_0805, F.Cu at (141.2, 110.0)
- added R12: 10kΩ, PCM_JLCPCB:R_0805, F.Cu at (137.8, 110.0)
- added R13: 18kΩ, PCM_JLCPCB:R_0603, F.Cu at (141.2, 125.0)
- added R14: 10kΩ, PCM_JLCPCB:R_0805, F.Cu at (141.2, 123.0)
- added R15: 100Ω, PCM_JLCPCB:R_0805, F.Cu at (141.2, 112.6)
- added R16: 10kΩ, PCM_JLCPCB:R_0805, F.Cu at (137.8, 112.6)
- added R17: 18kΩ, PCM_JLCPCB:R_0603, F.Cu at (139.0, 130.5)
- added R18: 10kΩ, PCM_JLCPCB:R_0805, F.Cu at (141.2, 127.0)
- added R19: 10kΩ, PCM_JLCPCB:R_0805, F.Cu at (134.8, 88.8)
- added R2: 10kΩ, PCM_JLCPCB:R_0603, F.Cu at (153.0, 137.5)
- added R20: 1kΩ, PCM_JLCPCB:R_0805, F.Cu at (125.0, 90.8)
- added R21: 470Ω, PCM_JLCPCB:R_0402, F.Cu at (119.5, 85.6)
- added R22: 1kΩ, PCM_JLCPCB:R_0805, F.Cu at (159.0, 120.6)
- added R23: 22kΩ, PCM_JLCPCB:R_0805, F.Cu at (157.0, 157.3)
- added R24: 10kΩ, PCM_JLCPCB:R_0805, F.Cu at (157.0, 153.7)
- added R25: 10kΩ, PCM_JLCPCB:R_0805, F.Cu at (159.1, 122.6)
- added R26: 33Ω, PCM_JLCPCB:R_0402, F.Cu at (142.4, 101.2)
- added R27: 10kΩ, PCM_JLCPCB:R_0805, F.Cu at (125.0, 93.8)
- added R28: 33Ω, PCM_JLCPCB:R_0402, F.Cu at (132.0, 98.6)
- added R29: 10kΩ, PCM_JLCPCB:R_0805, F.Cu at (134.5, 86.2)
- added R3: 100Ω, PCM_JLCPCB:R_0805, F.Cu at (141.2, 105.0)
- added R30: 33Ω, PCM_JLCPCB:R_0402, F.Cu at (139.0, 97.2)
- added R31: 33Ω, PCM_JLCPCB:R_0402, F.Cu at (135.2, 84.2)
- added R32: 33Ω, PCM_JLCPCB:R_0402, F.Cu at (124.6, 79.2)
- added R35: 33Ω, PCM_JLCPCB:R_0402, F.Cu at (132.0, 111.0)
- added R36: 33Ω, PCM_JLCPCB:R_0402, F.Cu at (132.0, 113.4)
- added R4: 10kΩ, PCM_JLCPCB:R_0805, F.Cu at (137.8, 105.0)
- added R5: 18kΩ, PCM_JLCPCB:R_0603, F.Cu at (141.0, 117.0)
- added R6: 10kΩ, PCM_JLCPCB:R_0805, F.Cu at (141.2, 115.0)
- added R7: 100Ω, PCM_JLCPCB:R_0805, F.Cu at (141.2, 107.4)
- added R8: 10kΩ, PCM_JLCPCB:R_0805, F.Cu at (137.8, 107.4)
- added R9: 18kΩ, PCM_JLCPCB:R_0603, F.Cu at (141.2, 121.0)
- added REF**: MountingHole_M3_7mm_Keepout, M3MountingHole:MountingHole_M3_7mm_Keepout, F.Cu at (159.2, 69.6)
- added REF**: MountingHole_M3_7mm_Keepout, M3MountingHole:MountingHole_M3_7mm_Keepout, F.Cu at (116.4, 69.6)
- added REF**: MountingHole_M3_7mm_Keepout, M3MountingHole:MountingHole_M3_7mm_Keepout, F.Cu at (116.4, 162.4)
- added REF**: MountingHole_M3_7mm_Keepout, M3MountingHole:MountingHole_M3_7mm_Keepout, F.Cu at (159.2, 162.4)
- added U1: TPS563201, Package_TO_SOT_SMD:SOT-23-6, F.Cu at (149.2, 144.8)
- added U4: ICM-42688-PC, Package_LGA:LGA-14_3x2.5mm_P0.5mm_LayoutBorder3x4y, F.Cu at (138.4, 85.6)
- added U5: MS5611-01BA, Package_LGA:LGA-8_3x5mm_P1.25mm, F.Cu at (122.1, 78.4)
- added U6: KX134-1211, KX134-1211:KIONIX_KXTJ3-1057, F.Cu at (136.7, 98.0)
Routing:
- net +5V: track 0.00 -> 213.2 mm
- net GND: track 0.00 -> 136.4 mm, vias 0 -> 89
- net /Flight Computer/RecoveryBuzzPower: track 0.00 -> 84.5 mm
- net /Flight Computer/Vbatt_Monitor: track 0.00 -> 79.6 mm, vias 0 -> 2
- net +8.4V_ARMED: track 0.00 -> 77.8 mm, vias 0 -> 15
- net /Flight Computer/Recovery_Buzzer: track 0.00 -> 70.2 mm, vias 0 -> 1
- net Net-(U1-SW): track 0.00 -> 68.0 mm, vias 0 -> 9
- net /Flight Computer/ServoPWM1: track 0.00 -> 58.9 mm
- net /Flight Computer/ServoPWM0: track 0.00 -> 58.9 mm
- net /Flight Computer/ServoPWM3: track 0.00 -> 54.2 mm
- net /Flight Computer/ServoPWM2: track 0.00 -> 53.9 mm
- net Net-(Q4-G): track 0.00 -> 47.2 mm, vias 0 -> 2
- net /Flight Computer/SCK1: track 0.00 -> 44.6 mm
- net /High-Power Actuators/Pyro2-: track 0.00 -> 44.4 mm
- net /High-Power Actuators/Pyro3-: track 0.00 -> 43.6 mm, vias 0 -> 2
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- added copper zone on In2.Cu, net +3.3V
- added copper zone on In2.Cu, net +8.4V_ARMED
- added copper zone on F.Cu, net GND
- added copper zone on In1.Cu, net GND
Other:
- board outline added: 50 x 100 mm
- copper layers 2 -> 4
- board text added: "+"
- board text added: "-"
- board text added: "ARM"
- board text added: "Detect Conn"
- board text added: "GND"
- board text added: "GX-12-4"
- board text added: "PY0"
- board text added: "PY1"
- board text added: "PY2"
- board text added: "PY3"
- board text added: "Prometheus Rocket Project Pronoia Flight Computer v1.0; 3/26"
- board text added: "Recov Buzz"
- board text added: "Rx"
- board text added: "S"
- board text added: "Tx"
- board text added: "UI Buzz"
- board text added: "UI LED"
